File: H-Bridge_Discrete.kicad_pcb (KiCad board)
At the start: 2 copper layers, 41 parts, among them J1 Conn_01x04, J2 Screw_Terminal_01x02, J3 Screw_Terminal_01x02, Q1 Q_NPN_EBC, Q10 Q_NMOS_GDS, Q11 Q_NPN_EBC, Q12 Q_PNP_EBC, Q13 Q_NPN_EBC, Q14 Q_PNP_EBC, Q15 Q_NPN_EBC, Q16 Q_NPN_EBC, Q2 Q_NPN_EBC, Q3 Q_NPN_EBC, Q4 Q_PNP_EBC, Q5 Q_NPN_EBC, Q6 Q_PNP_EBC, Q7 Q_NMOS_GDS, Q8 Q_NMOS_GDS, Q9 Q_NMOS_GDS

Commit message: 1
Parts:
- moved J2 30.6 mm to (55.9, 61.4)
- moved J1 30.6 mm to (55.2, 86.4)
- moved J3 28.3 mm to (142.9, 80.6)
- moved Q10 27.6 mm to (127.6, 111.8)
- moved Q9 21.3 mm to (127.6, 92.1)
- moved R7 18.5 mm to (136.5, 89.5)
- moved C1 18.3 mm to (55.2, 44.5)
- moved Q8 17.7 mm to (127.6, 71.8)
- moved Q7 17.7 mm to (127.6, 52.1)
- moved Q15 12.1 mm to (90.2, 124.5)
- moved R8 12.1 mm to (81.3, 110.5)
- moved C7 12.1 mm to (64.8, 127.0)
- moved Q11 12.1 mm to (103.5, 114.9)
- moved R10 12.1 mm to (81.3, 116.8)
- moved R11 12.1 mm to (73.0, 127.0)
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Routing:
- net SIG_A: track 135.4 -> 87.2 mm
- net SIG_B: track 102.5 -> 60.4 mm
- net Net-(Q13-Pad1): track 53.3 -> 33.5 mm
- net Net-(Q10-Pad1): track 53.9 -> 36.2 mm
- net Net-(Q5-Pad1): track 53.6 -> 36.5 mm
- net OUT_A: track 51.2 -> 34.9 mm
- net OUT_B: track 51.2 -> 35.1 mm
- net Net-(Q3-Pad1): track 51.7 -> 37.0 mm

Commit message: 1
Routing:
- added copper zone on B.Cu, net +12V
- added copper zone on F.Cu, net GND
- removed copper zone on F.Cu, net +12V
- removed copper zone on B.Cu, net GND

Commit message: 1
Parts:
- added REF**: SolderWire-2sqmm_1x01_D2mm_OD3.9mm, Connector_Wire:SolderWire-2sqmm_1x01_D2mm_OD3.9mm, F.Cu at (121.9, 50.8)
- added REF**: SolderWire-2sqmm_1x01_D2mm_OD3.9mm, Connector_Wire:SolderWire-2sqmm_1x01_D2mm_OD3.9mm, F.Cu at (121.9, 93.5)
- added REF**: SolderWire-2sqmm_1x01_D2mm_OD3.9mm, Connector_Wire:SolderWire-2sqmm_1x01_D2mm_OD3.9mm, F.Cu at (127.0, 122.9)
- added REF**: SolderWire-2sqmm_1x01_D2mm_OD3.9mm, Connector_Wire:SolderWire-2sqmm_1x01_D2mm_OD3.9mm, F.Cu at (127.0, 83.3)
- added REF**: , Connector_Wire:SolderWire-2sqmm_1x01_D2mm_OD3.9mm, F.Cu at (142.7, 56.9)
- added REF**: , Connector_Wire:SolderWire-2sqmm_1x01_D2mm_OD3.9mm, F.Cu at (142.7, 51.3)
- added REF**: SolderWire-2sqmm_1x01_D2mm_OD3.9mm, Connector_Wire:SolderWire-2sqmm_1x01_D2mm_OD3.9mm, F.Cu at (129.0, 45.2)
- added REF**: , Connector_Wire:SolderWire-2sqmm_1x01_D2mm_OD3.9mm, F.Cu at (135.1, 51.3)
- moved J2 88.5 mm to (142.9, 45.2), turned to 180 degrees
- moved C1 68.4 mm to (116.8, 74.2)
- moved R6 8.99 mm to (87.9, 69.6)
- moved C3 8.03 mm to (69.3, 53.6)
- moved D1 8.03 mm to (78.9, 47.9)
- moved R2 7.56 mm to (76.7, 53.6)
- moved Q1 7.08 mm to (92.7, 61.2)
- moved R1 7.08 mm to (83.8, 53.6)
- moved R5 7.08 mm to (83.8, 47.9)
- moved R8 6.65 mm to (87.9, 111.3)
- moved C5 6.48 mm to (115.3, 55.4)
- moved J1 5.72 mm to (61.0, 86.4)
- moved C7 5.49 mm to (69.3, 124.0)
- moved Q11 5.49 mm to (108.1, 111.9)
- moved Q12 5.49 mm to (108.1, 122.7)
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Routing:
- net SIG_A: track 87.2 -> 74.8 mm
- net Net-(C5-Pad1): track 62.2 -> 55.3 mm
- net Net-(C6-Pad1): track 62.2 -> 55.3 mm
- net Net-(Q10-Pad1): track 36.2 -> 30.4 mm
- net Net-(Q5-Pad1): track 36.5 -> 31.1 mm
- net SIG_B: track 60.4 -> 56.1 mm
- net Net-(Q2-Pad3): track 31.0 -> 27.8 mm
- net Net-(Q11-Pad2): track 31.0 -> 28.0 mm
- net OUT_A: track 34.9 -> 32.6 mm
- net Net-(Q3-Pad1): track 37.0 -> 34.8 mm
- net OUT_B: track 35.1 -> 33.3 mm
- net Net-(C8-Pad1): track 32.8 -> 31.5 mm
- net Net-(C3-Pad1): track 32.8 -> 31.5 mm
- net Net-(Q1-Pad3): track 28.5 -> 27.2 mm
- net Net-(Q13-Pad2): track 28.5 -> 27.5 mm
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- added copper zone on B.Cu, net GND
